Commit message: Updates as I try to get this to work with gazebo.

File: four_wheel_steering_controller/test/urdf/chassis.xacro (robot description, xacro)
@@ -3,12 +3,24 @@
   <!-- Base Properties -->
   <xacro:property name="mass_base" value="340" />
-  <xacro:property name="base_x_size" value="1.66000" />
-  <xacro:property name="base_y_size" value="0.60000" />
+  <xacro:property name="base_x_size" value="1.8000" />
+  <xacro:property name="base_y_size" value="1.80000" />
   <xacro:property name="base_z_size" value="0.66000" />
-  <xacro:property name="wheelbase" value="1.9" />
-  <xacro:property name="track" value="1.1" />
+  <xacro:property name="wheelbase" value="2" />
+  <xacro:property name="track" value="2" />
   <xacro:macro name="chassis">
     <!-- Base footprint is on the ground under the robot -->
-    <link name="base_footprint"/>
+    <gazebo reference="base_footprint">
+      <material>Gazebo/Grey</material>
+    </gazebo>
+    <link name="base_footprint">
+    <inertial>
+      <origin xyz="0 0 1" rpy="0 0 0"/>
+      <mass value="1"/>
+      <inertia
+        ixx="100.0" ixy="10.0" ixz="10.0"
+        iyy="100.0" iyz="10.0"
+        izz="100.0"/>
+    </inertial>
+    </link>
     <gazebo reference="base_link">
       <material>Gazebo/Grey</material>
@@ -16,4 +28,11 @@
     <!-- Base link is the center of the robot's bottom plate -->
     <link name="base_link">
+      <inertial>
+        <mass value="340" />
+        <origin xyz="0 0 0" />
+        <inertia ixx="${mass_base/12.0 * (base_y_size*base_y_size + base_z_size*base_z_size)}" ixy="1" ixz="1"
+                 iyy="${mass_base/12.0 * (base_x_size*base_x_size + base_z_size*base_z_size)}" iyz="1"
+                 izz="${mass_base/12.0 * (base_y_size*base_y_size + base_x_size*base_x_size)}" />
+      </inertial>
       <visual>
         <origin xyz="0 0 0" rpy="0 0 0" />
@@ -36,19 +55,4 @@
       <parent link="base_footprint" />
     </joint>
-    <!-- Interial link stores the robot's inertial information -->
-    <link name="inertial_link">
-      <inertial>
-        <mass value="340" />
-        <origin xyz="0 0 0" />
-        <inertia ixx="${mass_base/12.0 * (base_y_size*base_y_size + base_z_size*base_z_size)}" ixy="0" ixz="0"
-                 iyy="${mass_base/12.0 * (base_x_size*base_x_size + base_z_size*base_z_size)}" iyz="0"
-                 izz="${mass_base/12.0 * (base_y_size*base_y_size + base_x_size*base_x_size)}" />
-      </inertial>
-    </link>
-    <joint name="inertial_joint" type="fixed">
-      <origin xyz="0 0 0" rpy="0 0 0" />
-      <parent link="base_link" />
-      <child link="inertial_link" />
-    </joint>
   </xacro:macro>
 </robot>

File: four_wheel_steering_controller/test/urdf/four_wheel_steering.urdf.xacro (robot description, xacro)
@@ -5,7 +5,7 @@
   <xacro:property name="M_PI" value="3.14159"/>
   <!-- Wheel Mounting Positions -->
-  <xacro:property name="ground_clearance" value="0.19" />
-  <xacro:property name="wheel_x_offset" value="0.0" />
-  <xacro:property name="wheel_y_offset" value="0.05" />
+  <xacro:property name="ground_clearance" value="0.5" />
+  <xacro:property name="wheel_x_offset" value="0.001" />
+  <xacro:property name="wheel_y_offset" value="0.001" />
   <xacro:chassis/>
   <!-- Wheel macros -->
@@ -24,5 +24,9 @@
   <!-- Gazebo plugin for ROS Control -->
   <gazebo>
-    <plugin name="gazebo_ros_control" filename="libgazebo_ros_control.so"/>
+    <plugin name="gazebo_ros_control" filename="libgazebo_ros_control.so">
+    <legacyModeNS>true</legacyModeNS>
+    <robotNamespace>/</robotNamespace>
+    <robotSimType>gazebo_ros_control/DefaultRobotHWSim</robotSimType>
+  </plugin>
   </gazebo>
 </robot>

File: four_wheel_steering_controller/test/urdf/wheel.xacro (robot description, xacro)
@@ -4,6 +4,6 @@
   <!-- Wheel Properties -->
   <xacro:property name="wheel_length" value="0.1" />
-  <xacro:property name="wheel_radius" value="0.28" />
-  <xacro:property name="mass_wheel" value="5.0" />
+  <xacro:property name="wheel_radius" value="0.4" />
+  <xacro:property name="mass_wheel" value="500.0" />
   <xacro:macro name="wheel" params="wheel_prefix parent_link left_right *joint_origin">
     <gazebo reference="${wheel_prefix}_wheel_link">
@@ -56,5 +56,5 @@
 			</actuator>
 			<joint name="${wheel_prefix}_wheel">
-				<hardwareInterface>VelocityJointInterface</hardwareInterface>
+				<hardwareInterface>hardware_interface/VelocityJointInterface</hardwareInterface>
 			</joint>
 		</transmission>

File: four_wheel_steering_controller/test/urdf/wheel_steered.xacro (robot description, xacro)
@@ -3,5 +3,5 @@
   <xacro:property name="steering_link_y" value="0.05" />
   <xacro:property name="steering_link_xz" value="0.1" />
-  <xacro:property name="steering_link_mass" value="5.0" />
+  <xacro:property name="steering_link_mass" value="500.0" />
   <xacro:include filename="$(find four_wheel_steering_controller)/test/urdf/wheel.xacro" />
   <xacro:macro name="wheel_steered" params="wheel_prefix parent_link wheel_origin_y left_right *joint_origin ">
@@ -38,9 +38,9 @@
       <type>transmission_interface/SimpleTransmission</type>
       <actuator name="${wheel_prefix}_steering_motor">
-        <hardwareInterface>PositionJointInterface</hardwareInterface>
+        <hardwareInterface>hardware_interface/PositionJointInterface</hardwareInterface>
         <mechanicalReduction>1</mechanicalReduction>
       </actuator>
       <joint name="${wheel_prefix}_steering_joint">
-        <hardwareInterface>PositionJointInterface</hardwareInterface>
+        <hardwareInterface>hardware_interface/PositionJointInterface</hardwareInterface>
       </joint>
     </transmission>
